File: hardware/OpenRX-Lite.kicad_pcb (KiCad board)
At the start: 6 copper layers, 10 x 11.5 mm, 47 parts, among them U1 ESP32-C3, U2 TLV75533PDQNR, U3 SX1281IMLTRT, X1 CJ17-400001010B20

Commit message: Apply DroneAid rebrand and configure upstream sync
Other:
- board text added: "DroneAid"
- board text removed: "open"
